File: pad.kicad_sch (KiCad schematic)
At the start: 42 parts, among them U1 ADA4610-4xR, U2 ULN2002, U3 LP2901D

Commit message: Update schematic with some footprinit
Parts:
- JP10, JP20, JP30, JP40: footprint Jumper:SolderJumper-2_P1.3mm_Bridged2Bar_Pad1.0x1.5mm -> Jumper:SolderJumper-2_P1.3mm_Bridged2Bar_RoundedPad1.0x1.5mm
- R1, R10, R11, R2, R20, R21, R3, R30, R31, R4, R40, R41: footprint (none) -> Resistor_SMD:R_1210_3225Metric_Pad1.30x2.65mm_HandSolder
- TP1, TP11, TP13, TP14, TP15, TP3, TP4, TP5, TP6, TP7, TP8: footprint (none) -> TestPoint:TestPoint_Loop_D2.50mm_Drill1.85mm
- U2: footprint (none) -> External:SOIC127P600X175-16N

Commit message: Add push button on the footprint
Parts:
- A1: renamed from A; footprint (none) -> pad-button:button_A
- B1: renamed from B; footprint (none) -> pad-button:button_A
- C1: renamed from C; footprint (none) -> pad-button:button_A
- D1: renamed from D; footprint (none) -> pad-button:button_A
- Select1: renamed from Select; footprint (none) -> pad-button:button_start
- Start1: renamed from Start; footprint (none) -> pad-button:button_start
- TP12: footprint (none) -> TestPoint:TestPoint_Loop_D2.50mm_Drill1.85mm
Changed lines of the file:
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@@
   (symbol (lib_id "power:GND") (at 69.85 49.53 0) (unit 1)
     (in_bom yes) (on_board yes) (fields_autoplaced)
-    (property "Reference" "#PWR?" (id 0) (at 69.85 55.88 0)
+    (property "Reference" "#PWR0115" (id 0) (at 69.85 55.88 0)
       (effects (font (size 1.27 1.27)) hide)
     )
@@
   (symbol (lib_id "Switch:SW_Push") (at 190.5 100.33 0) (unit 1)
     (in_bom yes) (on_board yes) (fields_autoplaced)
-    (property "Reference" "Select" (id 0) (at 190.5 92.71 0))
+    (property "Reference" "Select1" (id 0) (at 190.5 92.71 0))
     (property "Value" "SW_Push" (id 1) (at 190.5 95.25 0))
-    (property "Footprint" "" (id 2) (at 190.5 95.25 0)
+    (property "Footprint" "pad-button:button_start" (id 2) (at 190.5 95.25 0)
       (effects (font (size 1.27 1.27)) hide)
     )
@@
   (symbol (lib_id "Switch:SW_Push") (at 190.5 110.49 0) (unit 1)
     (in_bom yes) (on_board yes) (fields_autoplaced)
-    (property "Reference" "A" (id 0) (at 190.5 102.87 0))
+    (property "Reference" "A1" (id 0) (at 190.5 102.87 0))
     (property "Value" "SW_Push" (id 1) (at 190.5 105.41 0))
-    (property "Footprint" "" (id 2) (at 190.5 105.41 0)
+    (property "Footprint" "pad-button:button_A" (id 2) (at 190.5 105.41 0)
       (effects (font (size 1.27 1.27)) hide)
     )
@@
   (symbol (lib_id "Switch:SW_Push") (at 190.5 120.65 0) (unit 1)
     (in_bom yes) (on_board yes) (fields_autoplaced)
-    (property "Reference" "B" (id 0) (at 190.5 113.03 0))
+    (property "Reference" "B1" (id 0) (at 190.5 113.03 0))
     (property "Value" "SW_Push" (id 1) (at 190.5 115.57 0))
-    (property "Footprint" "" (id 2) (at 190.5 115.57 0)
+    (property "Footprint" "pad-button:button_A" (id 2) (at 190.5 115.57 0)
       (effects (font (size 1.27 1.27)) hide)
     )
@@
       (effects (font (size 1.27 1.27)) (justify left))
     )
-    (property "Footprint" "" (id 2) (at 198.12 137.16 0)
+    (property "Footprint" "TestPoint:TestPoint_Loop_D2.50mm_Drill1.85mm" (id 2) (at 198.12 137.16 0)
       (effects (font (size 1.27 1.27)) hide)
     )
@@
   (symbol (lib_id "Switch:SW_Push") (at 190.5 90.17 0) (unit 1)
     (in_bom yes) (on_board yes) (fields_autoplaced)
-    (property "Reference" "Start" (id 0) (at 190.5 82.55 0))
+    (property "Reference" "Start1" (id 0) (at 190.5 82.55 0))
     (property "Value" "SW_Push" (id 1) (at 190.5 85.09 0))
-    (property "Footprint" "" (id 2) (at 190.5 85.09 0)
+    (property "Footprint" "pad-button:button_start" (id 2) (at 190.5 85.09 0)
       (effects (font (size 1.27 1.27)) hide)
     )
@@
   (symbol (lib_id "power:+5V") (at 58.42 29.21 0) (unit 1)
     (in_bom yes) (on_board yes) (fields_autoplaced)
-    (property "Reference" "#PWR?" (id 0) (at 58.42 33.02 0)
+    (property "Reference" "#PWR0114" (id 0) (at 58.42 33.02 0)
       (effects (font (size 1.27 1.27)) hide)
     )
@@
   (symbol (lib_id "Switch:SW_Push") (at 190.5 132.08 0) (unit 1)
     (in_bom yes) (on_board yes) (fields_autoplaced)
-    (property "Reference" "C" (id 0) (at 190.5 124.46 0))
+    (property "Reference" "C1" (id 0) (at 190.5 124.46 0))
     (property "Value" "SW_Push" (id 1) (at 190.5 127 0))
-    (property "Footprint" "" (id 2) (at 190.5 127 0)
+    (property "Footprint" "pad-button:button_A" (id 2) (at 190.5 127 0)
       (effects (font (size 1.27 1.27)) hide)
     )
@@
   (symbol (lib_id "power:GND") (at 58.42 49.53 0) (unit 1)
     (in_bom yes) (on_board yes) (fields_autoplaced)
-    (property "Reference" "#PWR?" (id 0) (at 58.42 55.88 0)
+    (property "Reference" "#PWR0116" (id 0) (at 58.42 55.88 0)
       (effects (font (size 1.27 1.27)) hide)
     )
@@
   (symbol (lib_id "Switch:SW_Push") (at 190.5 142.24 0) (unit 1)
     (in_bom yes) (on_board yes) (fields_autoplaced)
-    (property "Reference" "D" (id 0) (at 190.5 134.62 0))
+    (property "Reference" "D1" (id 0) (at 190.5 134.62 0))
     (property "Value" "SW_Push" (id 1) (at 190.5 137.16 0))
-    (property "Footprint" "" (id 2) (at 190.5 137.16 0)
+    (property "Footprint" "pad-button:button_A" (id 2) (at 190.5 137.16 0)
       (effects (font (size 1.27 1.27)) hide)
     )
@@
       (reference "#PWR0113") (unit 1) (value "+5V") (footprint "")
     )
+    (path "/caf849ae-e86d-4fa8-8dec-1ae24b642090"
+      (reference "#PWR0114") (unit 1) (value "+5V") (footprint "")
+    )
     (path "/061aaf97-97aa-4b05-a387-dbaf895cfd16"
-      (reference "#PWR?") (unit 1) (value "GND") (footprint "")
-    )
-    (path "/caf849ae-e86d-4fa8-8dec-1ae24b642090"
-      (reference "#PWR?") (unit 1) (value "+5V") (footprint "")
+      (reference "#PWR0115") (unit 1) (value "GND") (footprint "")
     )
     (path "/f1a2b3de-714f-410e-ad2c-656c181763cd"
-      (reference "#PWR?") (unit 1) (value "GND") (footprint "")
+      (reference "#PWR0116") (unit 1) (value "GND") (footprint "")
     )
     (path "/0e3c84cd-4ee3-456b-a593-8497e05d87a6"
-      (reference "A") (unit 1) (value "SW_Push") (footprint "")
+      (reference "A1") (unit 1) (value "SW_Push") (footprint "pad-button:button_A")
     )
     (path "/22045461-4478-4ac7-a8fe-7467bbc9a1ff"
-      (reference "B") (unit 1) (value "SW_Push") (footprint "")
+      (reference "B1") (unit 1) (value "SW_Push") (footprint "pad-button:button_A")
     )
     (path "/e5a0c5d3-4f35-4b65-8dd0-0e1999a40f2a"
-      (reference "C") (unit 1) (value "SW_Push") (footprint "")
+      (reference "C1") (unit 1) (value "SW_Push") (footprint "pad-button:button_A")
     )
     (path "/f9eeab6e-ab46-4639-97e0-11506a26da18"
-      (reference "D") (unit 1) (value "SW_Push") (footprint "")
+      (reference "D1") (unit 1) (value "SW_Push") (footprint "pad-button:button_A")
     )
     (path "/69453a36-dac6-4440-9a64-2ddb1e8a93e0"
@@
     )
     (path "/0970b113-13d6-449c-bc8b-5828314d144f"
-      (reference "Select") (unit 1) (value "SW_Push") (footprint "")
+      (reference "Select1") (unit 1) (value "SW_Push") (footprint "pad-button:button_start")
     )
     (path "/ab3d23f1-6526-43ab-815f-cf399fe2f53d"
-      (reference "Start") (unit 1) (value "SW_Push") (footprint "")
+      (reference "Start1") (unit 1) (value "SW_Push") (footprint "pad-button:button_start")
     )
     (path "/8f527890-0a50-4c70-b63a-e33b10defd7a"
@@
     )
     (path "/81b4d710-1c5f-4090-91dd-352ca975df9b"
-      (reference "TP12") (unit 1) (value "db15.12_ButtonC") (footprint "")
+      (reference "TP12") (unit 1) (value "db15.12_ButtonC") (footprint "TestPoint:TestPoint_Loop_D2.50mm_Drill1.85mm")
     )
     (path "/614d6e57-b339-4f9f-a330-2f819c6a8df6"

Commit message: Update schematic and board. All implemented, but not tested. Mechanical not tested yet
Parts:
- removed JP10, JP20, JP30, JP40: SolderJumper_2_Bridged, Jumper:SolderJumper-2_P1.3mm_Bridged2Bar_RoundedPad1.0x1.5mm, symbol Jumper:SolderJumper_2_Bridged
- removed JP11, JP21, JP31, JP41: SolderJumper_2_Open, Jumper:SolderJumper-2_P1.3mm_Open_RoundedPad1.0x1.5mm, symbol Jumper:SolderJumper_2_Open
- removed U3: LP2901D, Package_SO:SOIC-14_3.9x8.7mm_P1.27mm, symbol Comparator:LP2901D
- added C1, C11, C14, C15, C2, C21, C3, C31, C4, C41, C5, C6, C7: C, Capacitor_SMD:C_0603_1608Metric, symbol Device:C
- added R12, R22, R32, R42: R, Resistor_SMD:R_0603_1608Metric, symbol Device:R
- added U3: LM339, External:SOIC127P600X175-14N, symbol Comparator:LM339
- R10, R11, R20, R21, R30, R31, R40, R41: footprint Resistor_SMD:R_1210_3225Metric_Pad1.30x2.65mm_HandSolder -> Resistor_SMD:R_0603_1608Metric
- RV1: value x/y Axis -> RKJXV122400R; footprint (none) -> pad-button:RKJXV122400R_joystick
- TP1, TP11, TP12, TP13, TP14, TP15, TP3, TP4, TP5, TP6, TP7, TP8: footprint TestPoint:TestPoint_Loop_D2.50mm_Drill1.85mm -> TestPoint:TestPoint_Loop_D1.80mm_Drill1.0mm_Beaded
- U1: value ADA4610-4xR -> LPV324MX
- renumbered A1 to PB_A1, B1 to PB_B1, C1 to PB_C1, D1 to PB_D1, Select1 to PB_Select1, Start1 to PB_Start1
Connections:
- net +5V: now also C1.1, C2.1, C3.1, U3.3 (V+)
- net GND: now also C1.2, C11.2, C14.2, C15.2, C2.2, C21.2, C3.2, C31.2, C4.2, C41.2, C5.2, C6.2, C7.2, U3.12 (V-)
- net TP14_LEF: now also U2.14 (O3), C14.1, C41.1, R42.2
- net TP15_TOP: now also U2.15 (O2), C11.1, C15.1, R12.2
- net TP6_RIG: now also U2.13 (O4), C31.1, C6.1, R32.2
- net TP7_BOT: now also U2.16 (O1), C21.1, C7.1, R22.2
- net VRef_n: now also U3.7 (+), U3.9 (+)
- net VRef_p: now also U3.10 (-), U3.4 (-)
- net xAxis: now also C4.1, U3.5 (+), U3.6 (-)
- net yAxis: now also C5.1, U3.11 (+), U3.8 (-)
- new net: R22.1, U3.1
- new net: R12.1, U3.2
- new net: R42.1, U3.14
- new net: R32.1, U3.13
Other:
- note removed: "Comparator"
